File: output/pcbs/boardv3.kicad_pcb (KiCad board)
At the start: 2 copper layers, 167 x 122.9 mm, 67 parts

Commit message: release
Routing:
- net GND: track 107.3 -> 119.4 mm
Changed lines of the file:
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@@
   (segment (start 132.66 -7.04) (end 132.66 -4.37) (width 0.25) (layer "F.Cu") (net 42))
   (segment (start 126.7437 -15.8467) (end 127.2812 -16.3842) (width 0.25) (layer "F.Cu") (net 42))
+  (segment (start 114.4812 -12.7467) (end 113.1362 -14.0917) (width 0.25) (layer "F.Cu") (net 42))
+  (segment (start 117.7479 -17.78) (end 119.5812 -15.9467) (width 0.25) (layer "F.Cu") (net 42))
   (segment (start 114.8375 -12.3904) (end 114.4812 -12.7467) (width 0.25) (layer "F.Cu") (net 42))
   (segment (start 120.7563 -14.7716) (end 119.5812 -15.9467) (width 0.25) (layer "F.Cu") (net 42))
@@
   (segment (start 127.2812 -16.3842) (end 127.2812 -17.2119) (width 0.25) (layer "F.Cu") (net 42))
   (segment (start 125.4261 -45.3708) (end 123.5131 -45.3708) (width 0.25) (layer "F.Cu") (net 42))
+  (segment (start 113.1362 -16.6162) (end 114.3 -17.78) (width 0.25) (layer "F.Cu") (net 42))
+  (segment (start 113.1362 -14.0917) (end 113.1362 -16.6162) (width 0.25) (layer "F.Cu") (net 42))
+  (segment (start 114.3 -17.78) (end 117.7479 -17.78) (width 0.25) (layer "F.Cu") (net 42))
   (segment (start 126.7437 -15.8467) (end 126.2061 -15.8467) (width 0.25) (layer "F.Cu") (net 42))
   (via (at 132.66 -7.04) (size 0.8) (drill 0.4) (layers "F.Cu" "B.Cu") (net 42))
