File: ErgogenOutput/pcbs/boardv3.kicad_pcb (KiCad board)
At the start: 2 copper layers, 167 x 122.9 mm, 67 parts

Commit message: v4
Parts:
- removed B1, B2: , E73:SW_TACT_ALPS_SKQGABE010
- added ?: , , B.Cu at (164.9, 71.7)
- added ?: , , B.Cu at (166.6, 71.7)
- added ?: , , B.Cu at (166.6, 76.9)
- added ?: , , B.Cu at (164.9, 76.9)
- added REF**: Panasonic_EVQPUL_EVQPUC, Button_Switch_SMD:Panasonic_EVQPUL_EVQPUC, F.Cu at (165.7, 74.3)
- moved D1 82.9 mm to (34.3, 97.7)
- moved D2 82.9 mm to (34.3, 80.7)
- moved D28 82.9 mm to (152.7, 109.1)
- moved D29 82.9 mm to (164.8, 134.6)
- moved D3 82.9 mm to (34.3, 63.7)
- moved D4 82.9 mm to (34.3, 46.7)
- moved D5 82.9 mm to (53.3, 97.7)
- moved D6 82.9 mm to (53.3, 80.7)
- moved D7 82.9 mm to (53.3, 63.7)
- moved D8 82.9 mm to (53.3, 46.7)
- moved S1 82.9 mm to (34.3, 92.7)
- moved S2 82.9 mm to (34.3, 75.7)
- moved S27 82.9 mm to (148.5, 120.4)
- moved S29 82.9 mm to (167.7, 130.5)
- moved S3 82.9 mm to (34.3, 58.7)
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Routing:
- net RST: track 87.8 -> 67.1 mm
- net GND: track 119.4 -> 117.2 mm

Commit message: dualside complete
Parts:
- removed OLED2: OLED, lib:OLED_headers
- added ?: , , F.Cu at (148.5, 61.5)
- added ?: , , F.Cu at (148.5, 62.5)
- added ?: , , B.Cu at (148.3, 61.5)
- added ?: , , B.Cu at (153.5, 62.5)
- added ?: , , B.Cu at (153.5, 61.5)
- added ?: , , B.Cu at (148.3, 62.5)
- added ?: , , B.Cu at (145.9, 62.5)
- added ?: , , B.Cu at (151.0, 62.5)
- added ?: , , F.Cu at (151.0, 61.5)
- added ?: , , B.Cu at (145.9, 61.5)
- added ?: , , B.Cu at (156.2, 61.5)
- added ?: , , B.Cu at (151.0, 61.5)
- added ?: , , B.Cu at (156.2, 62.5)
- added ?: , , F.Cu at (156.1, 61.5)
- added ?: , , F.Cu at (153.7, 62.5)
- added ?: , , F.Cu at (145.8, 61.5)
- added ?: , , F.Cu at (153.7, 61.5)
- added ?: , , F.Cu at (145.8, 62.5)
- added ?: , , F.Cu at (156.1, 62.5)
- added ?: , , F.Cu at (151.0, 62.5)
- added REF**: SolderJumper-2_P1.3mm_Open_TrianglePad1.0x1.5mm, Jumper:SolderJumper-2_P1.3mm_Open_TrianglePad1.0x1.5mm, F.Cu at (151.9, 72.3)
- added REF**: SolderJumper-2_P1.3mm_Open_TrianglePad1.0x1.5mm, Jumper:SolderJumper-2_P1.3mm_Open_TrianglePad1.0x1.5mm, B.Cu at (151.9, 72.3)
Connections:
- OLED1 pad 0: P1 -> (no net)
- OLED1 pad 1: GND -> (no net)
- OLED1 pad 2: VCC -> (no net)
- OLED1 pad 3: P2 -> (no net)
- OLED1 pad 4: P0 -> (no net)
Routing:
- net (no net): track 0.00 -> 18.8 mm
- net P2: track 49.6 -> 63.4 mm
- net RST: track 67.1 -> 79.7 mm
- net P0: track 71.2 -> 82.7 mm, vias 2 -> 3
- net VCC: track 38.6 -> 47.2 mm
- net GND: track 117.2 -> 121.0 mm, vias 2 -> 4
- net P1: track 61.5 -> 59.6 mm, vias 1 -> 2

Commit message: pnp
Parts:
- moved ? 0.25 mm to (166.3, 71.7)
- moved ? 0.25 mm to (166.3, 76.9)
- moved REF** 0.25 mm to (165.5, 74.3)
- moved ? 0.25 mm to (164.6, 71.7)
- moved ? 0.25 mm to (164.6, 76.9)
Connections:
- REF** pad : (no net) -> RST
Routing:
- net RST: track 79.7 -> 81.0 mm
