File: pnp/pcbs/board.kicad_pcb (KiCad board)
At the start: 2 copper layers, 161.4 x 156.2 mm, 236 parts

Commit message: pnp
Parts:
- removed D100, D101, D102, D103, D104, D105, D106, D107, D108, D109, D110, D111, D112, D113, D114, D115, D116, D30, D32, D33, D35, D38, D39, D40, D42, D43, D44, D45, D46, D47, D48, D50, D55, D56, D60, D63, D65, D66, D70, D78, D80, D81, D82, D83, D86, D87, D88, D89, D90, D91, D92, D93, D94, D95, D96, D97, D98, D99: , ComboDiode
- removed the JST1 at (113.5, 1.42)
- removed the MCU1 at (126.6, -20.4)
- removed the OLED1 at (113.9, -2.09)
- removed S100, S101, S102, S103, S104, S105, S106, S107, S108, S109, S110, S111, S112, S113, S114, S115, S116, S88, S89, S90, S91, S92, S93, S94, S95, S96, S97, S98, S99: , PG1350
- removed the T1 at (127.5, 32.1)
- added JST1: , JST_PH_S2B-PH-K_02x2.00mm_Angled, F.Cu at (224.3, 56.7)
- added JST1: , JST_PH_S2B-PH-K_02x2.00mm_Angled, F.Cu at (137.7, 56.7)
- added MCU1: , ProMicro, F.Cu at (144.7, 32.2)
- added MCU1: , ProMicro, F.Cu at (217.3, 32.2)
- added OLED1: OLED, lib:OLED_headers, F.Cu at (137.2, 53.2)
- added OLED1: OLED, lib:OLED_headers, F.Cu at (210.3, 53.2)
- added Panasonic_EVQPUL_EVQPUC: Panasonic_EVQPUL_EVQPUC, Button_Switch_SMD:Panasonic_EVQPUL_EVQPUC, F.Cu at (203.1, 66.2)
- added Panasonic_EVQPUL_EVQPUC: Panasonic_EVQPUL_EVQPUC, Button_Switch_SMD:Panasonic_EVQPUL_EVQPUC, F.Cu at (159.0, 66.2)
- added T1: , E73:SPDT_C128955, F.Cu at (202.8, 82.7)
- added T1: , E73:SPDT_C128955, F.Cu at (159.2, 82.7)
- D1, D10, D11, D12, D13, D14, D15, D16, D17, D18, D19, D2, D20, D21, D22, D23, D24, D25, D26, D27, D28, D29, D3, D31, D34, D36, D37, D4, D41, D49, D5, D51, D52, D53, D54, D57, D58, D59, D6, D61, D62, D64, D67, D68, D69, D7, D71, D72, D73, D74, D75, D76, D77, D79, D8, D84, D85, D9: moved to B.Cu
- moved S33 95.6 mm to (334.3, 33.7), turned to 0 degrees
- moved S62 95.6 mm to (334.3, 33.7), turned to 0 degrees
- moved D62 95.1 mm to (334.3, 38.7), turned to 180 degrees
- moved S32 94.0 mm to (334.3, 50.7), turned to 0 degrees
- moved S61 94.0 mm to (334.3, 50.7), turned to 0 degrees
- moved D61 93.6 mm to (334.3, 55.7), turned to 180 degrees
- moved S31 92.6 mm to (334.3, 67.7), turned to 0 degrees
- moved S60 92.6 mm to (334.3, 67.7), turned to 0 degrees
- moved D31 92.2 mm to (334.3, 72.7), turned to 180 degrees
- moved S30 91.4 mm to (334.3, 84.7), turned to 0 degrees
- moved S59 91.4 mm to (334.3, 84.7), turned to 0 degrees
- moved D59 91.1 mm to (334.3, 89.7), turned to 180 degrees
- moved S37 91.0 mm to (315.3, 33.7), turned to 0 degrees
- moved S66 91.0 mm to (315.3, 33.7), turned to 0 degrees
- moved D37 90.5 mm to (315.3, 38.7), turned to 180 degrees
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Routing:
- net P20: track 0.00 -> 499.6 mm, vias 0 -> 1
- net P18: track 0.00 -> 427.5 mm, vias 0 -> 2
- net P19: track 0.00 -> 425.9 mm, vias 0 -> 1
- net P15: track 0.00 -> 393.6 mm
- net P14: track 0.00 -> 350.0 mm, vias 0 -> 1
- net P7: track 0.00 -> 319.2 mm
- net P3: track 0.00 -> 310.9 mm, vias 0 -> 2
- net P6: track 0.00 -> 292.3 mm
- net P5: track 0.00 -> 268.1 mm
- net P4: track 0.00 -> 254.0 mm
- net GND: track 0.00 -> 190.7 mm, vias 0 -> 1
- net P16: track 0.00 -> 151.0 mm, vias 0 -> 1
- net RAW: track 0.00 -> 146.0 mm, vias 0 -> 2
- net RST: track 0.00 -> 109.7 mm
- net P0: track 0.00 -> 88.5 mm
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Other:
- board size 161.4 x 156.2 mm -> 334.6 x 122.9 mm
- net class Default removed
