File: pnp/pcbs/pnpL.kicad_pcb (KiCad board)
At the start: 2 copper layers, 167 x 122.9 mm, 62 parts

Commit message: pnp
Parts:
- added Panasonic_EVQPUL_EVQPUC: Panasonic_EVQPUL_EVQPUC, Button_Switch_SMD:Panasonic_EVQPUL_EVQPUC, F.Cu at (159.4, 69.5)
- D1, D10, D11, D12, D13, D14, D15, D16, D17, D18, D19, D2, D20, D21, D22, D23, D24, D25, D26, D27, D28, D29, D3, D4, D5, D6, D7, D8, D9: moved to B.Cu
- turned D27 to 160 degrees
- turned D28 to 160 degrees
- turned D29 to 145 degrees
- turned D12 to 180 degrees
- turned D23 to 180 degrees
- turned D24 to 180 degrees
- turned D1 to 180 degrees
- turned D10 to 180 degrees
- turned D11 to 180 degrees
- turned D13 to 180 degrees
- turned D14 to 180 degrees
- turned D15 to 180 degrees
- turned D16 to 180 degrees
- turned D17 to 180 degrees
- turned D18 to 180 degrees
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Routing:
- net P20: track 0.00 -> 250.3 mm
- net P19: track 0.00 -> 209.1 mm, vias 0 -> 1
- net P18: track 0.00 -> 199.6 mm, vias 0 -> 1
- net P15: track 0.00 -> 183.7 mm
- net P7: track 0.00 -> 162.3 mm
- net P14: track 0.00 -> 162.3 mm
- net P3: track 0.00 -> 152.9 mm, vias 0 -> 1
- net P6: track 0.00 -> 149.7 mm
- net P5: track 0.00 -> 139.3 mm
- net P4: track 0.00 -> 133.4 mm
- net GND: track 0.00 -> 85.2 mm
- net RAW: track 0.00 -> 75.9 mm, vias 0 -> 1
- net RST: track 0.00 -> 61.5 mm
- net P16: track 0.00 -> 60.7 mm
- net P0: track 0.00 -> 41.4 mm
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