File: pnp/pcbs/pnpr.kicad_pcb (KiCad board)
At the start: 2 copper layers, 167 x 122.9 mm, 120 parts

Commit message: pnp
Parts:
- removed D30, D32, D33, D35, D38, D39, D40, D42, D43, D44, D45, D46, D47, D48, D50, D55, D56, D60, D63, D65, D66, D70, D78, D80, D81, D82, D83, D86, D87: , ComboDiode
- added Panasonic_EVQPUL_EVQPUC: Panasonic_EVQPUL_EVQPUC, Button_Switch_SMD:Panasonic_EVQPUL_EVQPUC, F.Cu at (38.4, 67.9)
- D31, D34, D36, D37, D41, D49, D51, D52, D53, D54, D57, D58, D59, D61, D62, D64, D67, D68, D69, D71, D72, D73, D74, D75, D76, D77, D79, D84, D85: moved to B.Cu
- turned D84 to 180 degrees
- turned D69 to 180 degrees
- turned D31 to 180 degrees
- turned D68 to 180 degrees
- turned D76 to 180 degrees
- turned D34 to 180 degrees
- turned D62 to 180 degrees
- turned D49 to 180 degrees
- turned D71 to 180 degrees
- turned D59 to 180 degrees
- turned D64 to 180 degrees
- turned D73 to 180 degrees
- turned D79 to 180 degrees
- turned D37 to 180 degrees
- turned D77 to 180 degrees
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Routing:
- net P20: track 0.00 -> 263.4 mm, vias 0 -> 1
- net P19: track 0.00 -> 240.0 mm
- net P18: track 0.00 -> 231.8 mm, vias 0 -> 1
- net P15: track 0.00 -> 210.1 mm
- net P14: track 0.00 -> 205.5 mm, vias 0 -> 1
- net P3: track 0.00 -> 158.0 mm, vias 0 -> 1
- net P7: track 0.00 -> 156.9 mm
- net P6: track 0.00 -> 142.6 mm
- net P5: track 0.00 -> 129.5 mm
- net P4: track 0.00 -> 120.6 mm
- net GND: track 0.00 -> 105.4 mm, vias 0 -> 1
- net P16: track 0.00 -> 90.3 mm, vias 0 -> 1
- net RAW: track 0.00 -> 70.1 mm, vias 0 -> 1
- net RST: track 0.00 -> 48.9 mm
- net P0: track 0.00 -> 47.1 mm
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